Commit message: about to write a subscriber fot the kinematics node

File: install/robotic_arm_description/share/robotic_arm_description/urdf/robotic_arm.xacro (robot description, xacro)
@@ -184,5 +184,5 @@
   <axis xyz="0.0 0.0 1.0"/>
   <dynamics damping="10.0" friction="2.0"/>
-  <limit upper="1.570796" lower="-1.570796" effort="100" velocity="100"/>
+  <limit upper="3.14" lower="-3.14" effort="100" velocity="100"/>
 </joint>
 <joint name="waist_link1_joint" type="revolute">
@@ -192,5 +192,5 @@
   <axis xyz="1.0 0.0 -0.0"/>
   <dynamics damping="10.0" friction="2.0"/>
-  <limit upper="1.570796" lower="-1.570796" effort="100" velocity="100"/>
+  <limit upper="3.14" lower="-3.14" effort="100" velocity="100"/>
 </joint>
 <joint name="link1_link2_joint" type="revolute">
@@ -200,5 +200,5 @@
   <axis xyz="-1.0 0.0 -0.0"/>
   <dynamics damping="10.0" friction="2.0"/>
-  <limit upper="3.141593" lower="0.0" effort="100" velocity="100"/>
+  <limit upper="3.14" lower="-3.14" effort="100" velocity="100"/>
 </joint>
 <joint name="link2_gripper_base_joint" type="revolute">
@@ -208,5 +208,5 @@
   <axis xyz="1.0 0.0 0.0"/>
   <dynamics damping="10.0" friction="2.0"/>
-  <limit upper="1.570796" lower="-1.570796" effort="100" velocity="100"/>
+  <limit upper="3.14" lower="-3.14" effort="100" velocity="100"/>
 </joint>
 <joint name="right_gripper_joint" type="revolute">

File: install/robotic_arm_moveit_config/share/robotic_arm_moveit_config/config/robotic_arm.ros2_control.xacro (robot description, xacro)
@@ -2,5 +2,5 @@
 <robot xmlns:xacro="http://www.ros.org/wiki/xacro">
     <xacro:macro name="robotic_arm_ros2_control" params="name initial_positions_file">
-        <xacro:property name="initial_positions" value="${xacro.load_yaml(initial_positions_file)['initial_positions']}"/>
+        <xacro:property name="initial_positions" value="${load_yaml(initial_positions_file)['initial_positions']}"/>
         <ros2_control name="${name}" type="system">
             <hardware>
